File: projects/Projeto 1 - Placa de Relé/Projeto 1 - Placa de Relé.kicad_pcb (KiCad board)
At the start: 2 copper layers, 35 x 55 mm, 8 parts, among them J1 Conn_01x03, J2 Screw_Terminal_01x03, K1 SRD-05VDC-SL-C, Q1 BC547

Commit message: chore: update project
Parts:
- moved J2 2.00 mm to (147.9, 132.0)
- moved J1 1.00 mm to (150.4, 89.0)
Routing:
- net /RL_COM: track 27.3 -> 25.2 mm
- net /RL_NC: track 13.4 -> 11.4 mm
- net /RL_NO: track 13.4 -> 11.4 mm
- net /SIG: track 18.3 -> 17.3 mm
Other:
- board text added: "5V"
- board text added: "COM"
- board text added: "GND"
- board text added: "NC"
- board text added: "NO"
- board text added: "Project: Relay Board Version: v1.0.0 Date: 05/10/2025"
- board text added: "S"
Changed lines of the file:
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@@
 		(tenting front back)
 		(pcbplotparams
-			(layerselection 0x00000000_00000000_55555555_5755f5ff)
+			(layerselection 0x00000000_00000000_55555555_57555554)
 			(plot_on_all_layers_selection 0x00000000_00000000_00000000_00000000)
 			(disableapertmacros no)
@@
 			(pdf_back_fp_property_popups yes)
 			(pdf_metadata yes)
-			(pdf_single_document no)
+			(pdf_single_document yes)
 			(dxfpolygonmode yes)
 			(dxfimperialunits yes)
@@
 			(crossoutdnponfab yes)
 			(subtractmaskfromsilk no)
-			(outputformat 1)
+			(outputformat 4)
 			(mirror no)
-			(drillshape 1)
+			(drillshape 2)
 			(scaleselection 1)
-			(outputdirectory "")
+			(outputdirectory "Projeto 1 - Placa de Relé-backups/outputs/pdf/")
 		)
 	)
@@
 	(footprint "Connector_PinHeader_2.54mm:PinHeader_1x03_P2.54mm_Vertical"
 		(layer "F.Cu")
-		(at 150.42 88 90)
+		(at 150.42 89 90)
 		(descr "Through hole straight pin header, 1x03, 2.54mm pitch, single row")
 		(tags "Through hole pin header THT 1x03 2.54mm single row")
@@
 		(tags "LED")
 		(property "Reference" "D1"
-			(at 1.27 -3.96 90)
+			(at -3.225 0 90)
 			(layer "F.SilkS")
 			(effects
@@
 		(tags "TO-92L Inline Wide transistor")
 		(property "Reference" "Q1"
-			(at 2.54 -3.56 90)
+			(at 7.04 0 180)
 			(layer "F.SilkS")
 			(effects
@@
 		(tags "Resistor Axial_DIN0207 series Axial Horizontal pin pitch 10.16mm 0.25W = 1/4W length 6.3mm diameter 2.5mm")
 		(property "Reference" "R1"
-			(at 5.08 -2.37 0)
+			(at 5.08 2.5 0)
 			(layer "F.SilkS")
 			(effects
@@
 	(footprint "TerminalBlock_Phoenix:TerminalBlock_Phoenix_MKDS-1,5-3-5.08_1x03_P5.08mm_Horizontal"
 		(layer "F.Cu")
-		(at 147.92 134)
+		(at 147.92 132)
 		(descr "Terminal Block Phoenix MKDS-1,5-3-5.08, 3 pins, pitch 5.08mm, size 15.2x9.8mm, drill diameter 1.3mm, pad diameter 2.6mm, http://www.farnell.com/datasheets/100425.pdf, script-generated using https://gitlab.com/kicad/libraries/kicad-footprint-generator/-/tree/master/scripts/TerminalBlock_Phoenix")
 		(tags "THT Terminal Block Phoenix MKDS-1,5-3-5.08 pitch 5.08mm size 15.2x9.8mm drill 1.3mm pad 2.6mm")
@@
 		(layer "Edge.Cuts")
 	)
+	(gr_text "S"
+		(at 152.5 87 0)
+		(layer "F.SilkS")
+		(effects
+			(font
+				(size 1 1)
+				(thickness 0.1)
+			)
+			(justify left bottom)
+		)
+	)
+	(gr_text "NC"
+		(at 157 139 0)
+		(layer "F.SilkS")
+		(effects
+			(font
+				(size 1 1)
+				(thickness 0.1)
+			)
+			(justify left bottom)
+		)
+	)
+	(gr_text "COM"
+		(at 151.452381 139 0)
+		(layer "F.SilkS")
+		(effects
+			(font
+				(size 1 1)
+				(thickness 0.1)
+			)
+			(justify left bottom)
+		)
+	)
+	(gr_text "5V"
+		(at 150.5 86.5 0)
+		(layer "F.SilkS")
+		(effects
+			(font
+				(size 1 1)
+				(thickness 0.125)
+			)
+		)
+	)
+	(gr_text "NO"
+		(at 147 139 0)
+		(layer "F.SilkS")
+		(effects
+			(font
+				(size 1 1)
+				(thickness 0.1)
+			)
+			(justify left bottom)
+		)
+	)
+	(gr_text "GND"
+		(at 154.5 87 0)
+		(layer "F.SilkS")
+		(effects
+			(font
+				(size 1 1)
+				(thickness 0.1)
+			)
+			(justify left bottom)
+		)
+	)
+	(gr_text "Project: Relay Board\nVersion: v1.0.0\nDate: 05/10/2025"
+		(at 167.5 122 90)
+		(layer "F.SilkS")
+		(effects
+			(font
+				(size 1 1)
+				(thickness 0.1)
+			)
+			(justify left bottom)
+		)
+	)
 	(segment
 		(start 164 97.265)
@@
 	)
 	(segment
-		(start 155.5 88)
-		(end 157.275 88)
-		(width 1)
-		(layer "B.Cu")
-		(net 2)
-	)
-	(segment
 		(start 141.5 94.96)
 		(end 145.96 94.96)
@@
 	)
 	(segment
-		(start 157.275 88)
+		(start 158.275 89)
 		(end 164 94.725)
+		(width 1)
+		(layer "B.Cu")
+		(net 2)
+	)
+	(segment
+		(start 155.5 89)
+		(end 158.275 89)
 		(width 1)
 		(layer "B.Cu")
@@
 	)
 	(segment
+		(start 137 94)
+		(end 142 89)
+		(width 1)
+		(layer "B.Cu")
+		(net 4)
+	)
+	(segment
 		(start 141.5 117.08)
 		(end 139.58 117.08)
@@
 	)
 	(segment
+		(start 142 89)
+		(end 150.42 89)
+		(width 1)
+		(layer "B.Cu")
+		(net 4)
+	)
+	(segment
+		(start 141.5 117.08)
+		(end 145.92 117.08)
+		(width 1)
+		(layer "B.Cu")
+		(net 4)
+	)
+	(segment
+		(start 137 114.5)
+		(end 137 94)
+		(width 1)
+		(layer "B.Cu")
+		(net 4)
+	)
+	(segment
+		(start 145.92 117.08)
+		(end 147.0675 115.9325)
+		(width 1)
+		(layer "B.Cu")
+		(net 4)
+	)
+	(segment
 		(start 139.58 117.08)
 		(end 137 114.5)
@@
 	)
 	(segment
-		(start 137 114.5)
-		(end 137 94)
-		(width 1)
-		(layer "B.Cu")
-		(net 4)
-	)
-	(segment
-		(start 143 88)
-		(end 150.42 88)
-		(width 1)
-		(layer "B.Cu")
-		(net 4)
-	)
-	(segment
-		(start 141.5 117.08)
-		(end 145.92 117.08)
-		(width 1)
-		(layer "B.Cu")
-		(net 4)
-	)
-	(segment
-		(start 137 94)
-		(end 143 88)
-		(width 1)
-		(layer "B.Cu")
-		(net 4)
-	)
-	(segment
-		(start 145.92 117.08)
-		(end 147.0675 115.9325)
-		(width 1)
-		(layer "B.Cu")
-		(net 4)
-	)
-	(segment
 		(start 158.16 99)
 		(end 158.16 97.74)
@@
 	(segment
 		(start 152.96 92.54)
-		(end 152.96 88)
+		(end 152.96 89)
 		(width 1.5)
 		(layer "B.Cu")
@@
 	)
 	(segment
-		(start 153.0675 133.9325)
-		(end 153 134)
-		(width 0.5)
-		(layer "F.Cu")
+		(start 153.0675 131.9325)
+		(end 153 132)
+		(width 2)
+		(layer "B.Cu")
 		(net 6)
 	)
 	(segment
-		(start 153.0675 133.9325)
-		(end 153 134)
-		(width 2)
-		(layer "B.Cu")
-		(net 6)
-	)
-	(segment
 		(start 153.0675 106.8)
-		(end 153.0675 133.9325)
+		(end 153.0675 131.9325)
 		(width 2)
 		(layer "B.Cu")
@@
 	(segment
 		(start 158.08 128.42)
-		(end 158.08 134)
+		(end 158.08 132)
 		(width 2)
 		(layer "B.Cu")
@@
 	)
 	(segment
+		(start 147.0675 121)
+		(end 147.0675 127.0675)
+		(width 2)
+		(layer "B.Cu")
+		(net 8)
+	)
+	(segment
+		(start 147.92 128.08)
+		(end 147.92 132)
+		(width 2)
+		(layer "B.Cu")
+		(net 8)
+	)
+	(segment
 		(start 147.0675 127.0675)
 		(end 148 128)
@@
 	)
 	(segment
-		(start 147.92 128.08)
-		(end 147.92 134)
-		(width 2)
-		(layer "B.Cu")
-		(net 8)
-	)
-	(segment
 		(start 148 128)
 		(end 147.92 128.08)
 		(width 2)
 		(layer "B.Cu")
-		(net 8)
-	)
-	(segment
-		(start 147.0675 121)
-		(end 147.0675 127.0675)
-		(width 2)
-		(layer "B.Cu")
