File: projects/Projeto 2 - Placa com microcontrolador/Projeto 2 - Placa com microcontrolador.kicad_sch (KiCad schematic)
At the start: 0 parts

Commit message: feat: add projects files
Other:
- added sheet 3.3V Regulator (3VRegulator.kicad_sch)
- added sheet Input 12V (Input12V.kicad_sch)
- added sheet Interface (Interface.kicad_sch)
- added sheet MCU (MCU.kicad_sch)
- added sheet Motor (Motor.kicad_sch)
Changed lines of the file:
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@@
 	(generator_version "9.0")
 	(paper "A4")
+	(sheet
+		(at 208.28 78.74)
+		(size 25.4 22.86)
+		(exclude_from_sim no)
+		(in_bom yes)
+		(on_board yes)
+		(dnp no)
+		(fields_autoplaced yes)
+		(stroke
+			(width 0.1524)
+			(type solid)
+		)
+		(fill
+			(color 0 0 0 0.0000)
+		)
+		(property "Sheetname" "Motor"
+			(at 208.28 78.0284 0)
+			(effects
+				(font
+					(size 1.27 1.27)
+				)
+				(justify left bottom)
+			)
+		)
+		(property "Sheetfile" "Motor.kicad_sch"
+			(at 208.28 102.1846 0)
+			(effects
+				(font
+					(size 1.27 1.27)
+				)
+				(justify left top)
+			)
+		)
+		(instances
+			(project "Projeto 2 - Placa com microcontrolador"
+				(path "/dd7c4082-b1f8-4aea-8c69-8cbf0854fd10"
+					(page "6")
+				)
+			)
+		)
+	)
+	(sheet
+		(at 67.31 78.74)
+		(size 22.86 22.86)
+		(exclude_from_sim no)
+		(in_bom yes)
+		(on_board yes)
+		(dnp no)
+		(fields_autoplaced yes)
+		(stroke
+			(width 0.1524)
+			(type solid)
+		)
+		(fill
+			(color 0 0 0 0.0000)
+		)
+		(property "Sheetname" "Input 12V"
+			(at 67.31 78.0284 0)
+			(effects
+				(font
+					(size 1.27 1.27)
+				)
+				(justify left bottom)
+			)
+		)
+		(property "Sheetfile" "Input12V.kicad_sch"
+			(at 67.31 102.1846 0)
+			(effects
+				(font
+					(size 1.27 1.27)
+				)
+				(justify left top)
+			)
+		)
+		(instances
+			(project "Projeto 2 - Placa com microcontrolador"
+				(path "/dd7c4082-b1f8-4aea-8c69-8cbf0854fd10"
+					(page "2")
+				)
+			)
+		)
+	)
+	(sheet
+		(at 104.14 78.74)
+		(size 22.86 22.86)
+		(exclude_from_sim no)
+		(in_bom yes)
+		(on_board yes)
+		(dnp no)
+		(fields_autoplaced yes)
+		(stroke
+			(width 0.1524)
+			(type solid)
+		)
+		(fill
+			(color 0 0 0 0.0000)
+		)
+		(property "Sheetname" "3.3V Regulator"
+			(at 104.14 78.0284 0)
+			(effects
+				(font
+					(size 1.27 1.27)
+				)
+				(justify left bottom)
+			)
+		)
+		(property "Sheetfile" "3VRegulator.kicad_sch"
+			(at 104.14 102.1846 0)
+			(effects
+				(font
+					(size 1.27 1.27)
+				)
+				(justify left top)
+			)
+		)
+		(instances
+			(project "Projeto 2 - Placa com microcontrolador"
+				(path "/dd7c4082-b1f8-4aea-8c69-8cbf0854fd10"
+					(page "3")
+				)
+			)
+		)
+	)
+	(sheet
+		(at 139.7 78.74)
+		(size 22.86 38.1)
+		(exclude_from_sim no)
+		(in_bom yes)
+		(on_board yes)
+		(dnp no)
+		(fields_autoplaced yes)
+		(stroke
+			(width 0.1524)
+			(type solid)
+		)
+		(fill
+			(color 0 0 0 0.0000)
+		)
+		(property "Sheetname" "MCU"
+			(at 139.7 78.0284 0)
+			(effects
+				(font
+					(size 1.27 1.27)
+				)
+				(justify left bottom)
+			)
+		)
+		(property "Sheetfile" "MCU.kicad_sch"
+			(at 139.7 117.4246 0)
+			(effects
+				(font
+					(size 1.27 1.27)
+				)
+				(justify left top)
+			)
+		)
+		(instances
+			(project "Projeto 2 - Placa com microcontrolador"
+				(path "/dd7c4082-b1f8-4aea-8c69-8cbf0854fd10"
+					(page "4")
+				)
+			)
+		)
+	)
+	(sheet
+		(at 173.99 78.74)
+		(size 24.13 22.86)
+		(exclude_from_sim no)
+		(in_bom yes)
+		(on_board yes)
+		(dnp no)
+		(fields_autoplaced yes)
+		(stroke
+			(width 0.1524)
+			(type solid)
+		)
+		(fill
+			(color 0 0 0 0.0000)
+		)
+		(property "Sheetname" "Interface"
+			(at 173.99 78.0284 0)
+			(effects
+				(font
+					(size 1.27 1.27)
+				)
+				(justify left bottom)
+			)
+		)
+		(property "Sheetfile" "Interface.kicad_sch"
+			(at 173.99 102.1846 0)
+			(effects
+				(font
+					(size 1.27 1.27)
+				)
+				(justify left top)
+			)
+		)
+		(instances
+			(project "Projeto 2 - Placa com microcontrolador"
+				(path "/dd7c4082-b1f8-4aea-8c69-8cbf0854fd10"
+					(page "5")
+				)
+			)
+		)
+	)
 	(sheet_instances
 		(path "/"
@@
 	)
 	(embedded_fonts no)
+	(embedded_files
+		(file
+			(name "sheet.kicad_wks")
+			(type worksheet)
+			(data |KLUv/WDpCc0UAHadXSEAtxsWHGS5ac4JWlhdTS3ZQeABkGbFFme+cSP//z/UEwFTAEwAWAD4H38k
+				/o/H5kn7Wk/2Rs53XDRg1Jr9+dCS/FrRgFm0/WTLL/kXAICAgBS9l9NaVJzKhs4Ryaozfi/7dY8h
+				o5Redda+2JbZRwVAQFCGSJzQA22oEH9xhzZWu8RkRav+kv/32Lyw2hMzlTJ47XtOes5+MwZf7Nmz
+				CoFY/NrFt9/++Q6vCGevq/7r44jB2rXD64irJ6X92fuyqtpH7z7oeQyXzaJZ/GQxoYi/RlROs11G
+				fsmyqiPUQvRiUkqFw1w2DcehNbgIioBZWE9KF1aiFVlq6zQHZ8tgMByK0Ax/z5FzNmX/62CbOvZL
+				EQirTTVTxXp+3zfpVQAEAYGhJiq2uOqFqIuLJuq8aEfZJqbrkSNuzLqhaJZJpaGAdJql2zYIJssu
+				CzHRKJuEe9gHaEXvbSusSTdJx3Xi267SSkPb7/7BDA6pQchV/d6Ycaezk54lgICg8USGGJoSKUiS
+				FDqARKTmqBvcLGt61Ov0GmN9RMp16OPryEhYdd4Zdt3vqhHCMTDPdX5jgtwaJiv8cnNZZHcy5Nsk
+				GXCbxZPwCdfFZSBOK8Ac05OTpyY7mxeSk+5jmuPyTxPzqQzuKUShJrG0XRjic3B4c1xZEh9gXxl+
+				1ABDm5/y2QTBJIwrCDDB8jQaql1KNUyWjVMH8QX9TybGpIUcNMOn7IkaBjTk9I++smxucthTblHX
+				XHppqw0FQrpz2hMFCt44iw9+c8x7tBWws7glWu74914ZttTgplcQCFL15JSApiaPMAYI8qdD+pQM
+				L3vRw+TVwOGgw6weLXO25ElCy3KytiHETfyGvUuvJjVN08b6bywPUXeZ60M6BqsK|
+			)
+			(checksum "E884C03FA7E5CAC04A971A43712DA87E")
+		)
+	)
 )
